Commit message: ok

File: src/ashwini/urdf/ashwini.xacro (robot description, xacro)
@@ -255,5 +255,5 @@
 			<origin xyz="0 0 0" rpy="0 0 0"/>
 			<geometry>
-				<mesh filename="package://atom/meshes/hokuyo.dae"/>
+				<mesh filename="package://ashwini/meshes/hokuyo.dae"/>
 			</geometry>
 		</visual>
